File: Eagle/mod2/TK90X.brd (EAGLE design)
At the start: 217.8 x 132.1 mm, 219 parts, among them IC1 Z80, IC10 74LS365N, IC11 LM1886, IC12 LM1889, IC13 4116, IC14 4116, IC15 4116, IC16 4116, IC17 4116, IC18 4116, IC19 4116, IC2 ROM, IC20 4116, IC21 4416, IC22 4416, IC23 4416, IC24 4416, IC25 74LS00, IC26 74LS00, IC27 74LS32, IC28 74LS04, IC3 ULA TK90, IC4 74LS74, IC5 74LS74, IC6 74LS157, IC7 74LS157, IC8 74LS157, IC9 74LS157, Q1 BC548, Q2 BC548, Q3 BF494, Q4 BC548, Q5 BD139, Q6 BD136, Q7 BC548, Q8 2N4401, X2 POWER

Commit message: Alguns ajustes no mod2
Parts:
- removed CVBS: RF, testpad:P1-13
- added X1: RCA2PINA1, tk90:TOBU3
- Q8: device transistor-npn:TO92 -> tk90:TO92-EBC
- moved C58 22.9 mm to (17.1, 127.6)
- moved R57 5.99 mm to (39.4, 113.7), turned to 270 degrees
- moved C43 5.12 mm to (52.7, 125.7), turned to 270 degrees
- moved R58 2.62 mm to (31.8, 122.6), turned to 270 degrees
- moved C41 2.54 mm to (31.8, 113.7)
- moved L3 2.54 mm to (35.6, 113.7)
Connections:
- removed net N$76: C58.-, CVBS.1
- new net N$74: C58.-, X1.PIN
- net +5V: now also Q8.C; no longer Q8.1
- net GND: now also X1.SHELL, X1.SHELL@1, X1.SHELL@2
- net N$48: now also Q8.E; no longer Q8.3
- net N$69: now also Q8.B; no longer Q8.2
Routing:
- net N$74: track 0.00 -> 28.1 mm
- net N$48: track 33.8 -> 10.8 mm
- net N$76: track 11.5 -> 0.00 mm
- net +12V: track 357.1 -> 367.1 mm
- net N$87: track 12.0 -> 13.6 mm
- net N$69: track 83.4 -> 82.8 mm
- net +5V: track 1051.5 -> 1052.1 mm
