File: Eagle/mod2/TK90X.sch (EAGLE design)
At the start: 219 parts, among them IC1 Z80, IC10 74LS365N, IC11 LM1886, IC12 LM1889, IC13 4116, IC14 4116, IC15 4116, IC16 4116, IC17 4116, IC18 4116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

Commit message: Alguns ajustes no mod2
Parts:
- removed CVBS: RF, testpad:TPPAD1-13
- added X1: RCA2PINA1, tk90:RCA2PINA1
- Q8: device transistor-npn:2N4416 -> tk90:2N4401
Connections:
- removed net N$76: C58.-, CVBS.TP
- new net N$74: C58.-, X1.1
- net GND: now also X1.2
Other:
- moved on the sheet: C58, R59
