File: Rev4/Eagle/TK90X.sch (EAGLE design)
At the start: 217 parts, among them IC1 Z80, IC10 74LS365N, IC11 LM1886, IC12 LM1889, IC13 4116, IC14 4116, IC15 4116, IC16 4116, IC17 4116, IC18 4116, IC19 4116, IC2 ROM, IC20 4116, IC21 4416, IC22 4416, IC23 4416, IC24 4416, IC25 74LS00, IC26 74LS00, IC27 74LS32, IC28 74LS04, IC3 ULA TK90, IC4 74LS74, IC5 74LS74, IC6 74LS157, IC7 74LS157, IC8 74LS157, IC9 74LS157, Q1 BC548, Q2 BC548, Q3 BF494, Q4 BC548, Q5 BD139, Q6 BD136, Q7 BC548, X2 POWER

Commit message: Corrigido conexões power Adicionado jumpers de solda pros jacks de áudio Adicionado revisão 6 com 74LS365 substituido pelo 74LS244
Parts:
- added J1, J2: 0R-JUMPB, jump-0r-smd:0R-JUMPB
- added J3: (no value), jumper:SJ
Connections:
- new net N$33: C26.1, C27.1, IC13.VBB, IC14.VBB, IC15.VBB, IC16.VBB, IC17.VBB, IC18.VBB, IC19.VBB, IC20.VBB, J3.2
- new net N$48: IC2.!PGM, J1-0R.2
- new net VDD: C23.1, C25.1, C28.1, C30.1, IC13.VDD, IC14.VDD, IC15.VDD, IC16.VDD, IC17.VDD, IC18.VDD, IC19.VDD, IC20.VDD, J2-0R.2
- net !RD: now also J1-0R.3; no longer IC2.!PGM
- net +5V: now also J1-0R.1, J2-0R.1
- net -5V: now also J3.1; no longer C26.1, C27.1, IC13.VBB, IC14.VBB, IC15.VBB, IC16.VBB, IC17.VBB, IC18.VBB, IC19.VBB, IC20.VBB
- net V+: now also J2-0R.3; no longer C23.1, C25.1, C28.1, C30.1, IC13.VDD, IC14.VDD, IC15.VDD, IC16.VDD, IC17.VDD, IC18.VDD, IC19.VDD, IC20.VDD
Other:
- note added: "FBLabs rev 4"
- note removed: "FBLabs rev 3"
- moved on the sheet: C26, C27
