File: Rev5/Eagle/TK90X.sch (EAGLE design)
At the start: 221 parts, among them IC1 Z80, IC10 74LS365N, IC11 LM1886, IC12 LM1889, IC13 4116, IC14 4116, IC15 4116, IC16 4116, IC17 4116, IC18 4116, IC19 4116, IC2 ROM, IC20 4116, IC21 4416, IC22 4416, IC23 4416, IC24 4416, IC25 74LS00, IC26 74LS00, IC27 74LS32, IC28 74LS04, IC3 ULA TK90, IC4 74LS74, IC5 74LS74, IC6 74LS157, IC7 74LS157, IC8 74LS157, IC9 74LS157, J1 0R-JUMPB, J2 0R-JUMPB, Q1 BC548, Q2 BC548, Q3 BF494, Q4 BC548, Q5 BD139, Q6 BD136, Q7 BC548, Q8 BC517, X1 RCA2PINA1, X2 POWER

Commit message: Corrigido conexões power Adicionado jumpers de solda pros jacks de áudio Adicionado revisão 6 com 74LS365 substituido pelo 74LS244
Parts:
- added J5: (no value), jumper:SJ
Connections:
- new net N$88: EAR.NC, J5.2
- net N$16: now also J5.1; no longer EAR.NC
- net V+: now also X2.NC
Other:
- note added: "FBLabs rev 5"
- moved on the sheet: EAR
Changed lines of the file:
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@@
 <part name="J1" library="jump-0r-smd" deviceset="0R-JUMP" device="B"/>
 <part name="P+46" library="supply1" deviceset="+5V" device=""/>
+<part name="J5" library="jumper" deviceset="SJ" device=""/>
 </parts>
 <sheets>
@@
 <text x="-414.02" y="96.52" size="1.778" layer="97" font="vector"># Diodos 1N4148 exceto Zeners (D21,D24)  e Varicap (D28)</text>
 <text x="-144.78" y="414.02" size="1.778" layer="96" rot="R90">8x1N4148</text>
+<text x="370.84" y="7.62" size="5.08" layer="97">FBLabs rev 5</text>
 </plain>
 <instances>
@@
 <attribute name="VALUE" x="-149.86" y="170.18" size="1.778" layer="96" rot="R180"/>
 </instance>
-<instance part="EAR" gate="G$1" x="-7.62" y="195.58" smashed="yes" rot="MR0">
-<attribute name="NAME" x="-5.08" y="199.644" size="1.778" layer="95" rot="MR0"/>
-<attribute name="VALUE" x="-7.62" y="191.008" size="1.778" layer="96" rot="MR180"/>
+<instance part="EAR" gate="G$1" x="20.32" y="195.58" smashed="yes" rot="MR0">
+<attribute name="NAME" x="22.86" y="199.644" size="1.778" layer="95" rot="MR0"/>
+<attribute name="VALUE" x="20.32" y="191.008" size="1.778" layer="96" rot="MR180"/>
 </instance>
 <instance part="R41" gate="G$1" x="-71.12" y="190.5" smashed="yes" rot="R90">
@@
 <instance part="GND21" gate="1" x="-22.86" y="182.88"/>
 <instance part="GND22" gate="1" x="-60.96" y="182.88"/>
-<instance part="GND23" gate="1" x="-10.16" y="182.88"/>
+<instance part="GND23" gate="1" x="17.78" y="182.88"/>
 <instance part="P+22" gate="1" x="-71.12" y="213.36" smashed="yes">
 <attribute name="VALUE" x="-73.66" y="213.36" size="1.778" layer="96" rot="R180"/>
@@
 <attribute name="VALUE" x="-330.2" y="330.2" size="1.778" layer="96" rot="R180"/>
 </instance>
+<instance part="J5" gate="1" x="2.54" y="195.58" smashed="yes">
+<attribute name="NAME" x="2.032" y="191.262" size="1.778" layer="95"/>
+<attribute name="VALUE" x="0" y="191.77" size="1.778" layer="96"/>
+</instance>
 </instances>
 <busses>
@@
 </segment>
 <segment>
-<wire x1="-10.16" y1="193.04" x2="-10.16" y2="185.42" width="0.1524" layer="91"/>
+<wire x1="17.78" y1="193.04" x2="17.78" y2="185.42" width="0.1524" layer="91"/>
 <pinref part="EAR" gate="G$1" pin="SHIELD"/>
 <pinref part="GND23" gate="1" pin="GND"/>
@@
 <net name="N$16" class="0">
 <segment>
-<wire x1="-10.16" y1="198.12" x2="-12.7" y2="198.12" width="0.1524" layer="91"/>
-<wire x1="-12.7" y1="198.12" x2="-22.86" y2="198.12" width="0.1524" layer="91"/>
+<wire x1="17.78" y1="198.12" x2="-5.08" y2="198.12" width="0.1524" layer="91"/>
+<wire x1="-5.08" y1="198.12" x2="-22.86" y2="198.12" width="0.1524" layer="91"/>
 <wire x1="-22.86" y1="198.12" x2="-22.86" y2="195.58" width="0.1524" layer="91"/>
 <wire x1="-30.48" y1="198.12" x2="-22.86" y2="198.12" width="0.1524" layer="91"/>
@@
 <pinref part="EAR" gate="G$1" pin="TIP"/>
 <pinref part="R70" gate="G$1" pin="2"/>
-<pinref part="EAR" gate="G$1" pin="NC"/>
-<wire x1="-10.16" y1="195.58" x2="-12.7" y2="195.58" width="0.1524" layer="91"/>
-<wire x1="-12.7" y1="195.58" x2="-12.7" y2="198.12" width="0.1524" layer="91"/>
-<junction x="-12.7" y="198.12"/>
 <pinref part="C5" gate="G$1" pin="-"/>
+<pinref part="J5" gate="1" pin="1"/>
+<wire x1="-2.54" y1="195.58" x2="-5.08" y2="195.58" width="0.1524" layer="91"/>
+<wire x1="-5.08" y1="195.58" x2="-5.08" y2="198.12" width="0.1524" layer="91"/>
+<junction x="-5.08" y="198.12"/>
 </segment>
 </net>
@@
 <wire x1="-381" y1="129.54" x2="-381" y2="134.62" width="0.1524" layer="91"/>
 <junction x="-381" y="134.62"/>
-<wire x1="-391.16" y1="134.62" x2="-381" y2="134.62" width="0.1524" layer="91"/>
+<wire x1="-391.16" y1="134.62" x2="-388.62" y2="134.62" width="0.1524" layer="91"/>
 <pinref part="P+42" gate="1" pin="V+"/>
+<wire x1="-388.62" y1="134.62" x2="-381" y2="134.62" width="0.1524" layer="91"/>
 <wire x1="-370.84" y1="137.16" x2="-370.84" y2="134.62" width="0.1524" layer="91"/>
 <pinref part="X2" gate="G$1" pin="TIP"/>
+<pinref part="X2" gate="G$1" pin="NC"/>
+<wire x1="-391.16" y1="132.08" x2="-388.62" y2="132.08" width="0.1524" layer="91"/>
+<wire x1="-388.62" y1="132.08" x2="-388.62" y2="134.62" width="0.1524" layer="91"/>
+<junction x="-388.62" y="134.62"/>
 </segment>
 </net>
@@
 </segment>
 </net>
+<net name="N$88" class="0">
+<segment>
+<pinref part="EAR" gate="G$1" pin="NC"/>
+<pinref part="J5" gate="1" pin="2"/>
+<wire x1="17.78" y1="195.58" x2="7.62" y2="195.58" width="0.1524" layer="91"/>
+</segment>
+</net>
