File: Rev6/Eagle/TK90X.brd (EAGLE design)
At the start: 217.8 x 132.1 mm, 221 parts, among them IC1 Z80, IC10 74LS244N, IC11 LM1886, IC12 LM1889, IC13 4116, IC14 4116, IC15 4116, IC16 4116, IC17 4116, IC18 4116, IC19 4116, IC2 ROM, IC20 4116, IC21 4416, IC22 4416, IC23 4416, IC24 4416, IC25 74LS00, IC26 74LS00, IC27 74LS32, IC28 74LS04, IC3 ULA TK90, IC4 74LS74, IC5 74LS74, IC6 74LS157, IC7 74LS157, IC8 74LS157, IC9 74LS157, J1 0R-JUMPB, J2 0R-JUMPB, Q1 BC548, Q2 BC548, Q3 BF494, Q4 BC548, Q5 BD139, Q6 BD136, Q7 BC548, Q8 BC517, X1 RCA2PINN1, X2 POWER

Commit message: Corrigido valores de R68 e C52 para melhor geração dos 12V para o Vídeo e DRAMs. Corrigido largura de algumas trilhas
Parts:
- C52: value 1u -> 10u
- R68: value 100 -> 33
Changed lines of the file:
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@@
 <attribute name="VALUE" x="14.5415" y="55.0545" size="1.27" layer="27" ratio="10" rot="R180"/>
 </element>
-<element name="C52" library="rcl" package="E2-5" value="1u" x="6.0325" y="93.6625" smashed="yes" rot="R90">
+<element name="C52" library="rcl" package="E2-5" value="10u" x="6.0325" y="93.6625" smashed="yes" rot="R90">
 <attribute name="NAME" x="4.445" y="96.5835" size="1.27" layer="25" ratio="10"/>
 <attribute name="VALUE" x="2.8575" y="90.2335" size="1.27" layer="27" ratio="10"/>
@@
 <attribute name="VALUE" x="7.0358" y="41.529" size="1.27" layer="27" ratio="10" rot="R90"/>
 </element>
-<element name="R68" library="rcl" package="0207/12" value="100" x="9.525" y="73.66" smashed="yes" rot="R90">
+<element name="R68" library="rcl" package="0207/12" value="33" x="9.525" y="73.66" smashed="yes" rot="R90">
 <attribute name="NAME" x="8.763" y="76.835" size="1.27" layer="25" ratio="10" rot="R90"/>
 <attribute name="VALUE" x="10.2108" y="72.3265" size="1.27" layer="27" ratio="10" rot="R90"/>
@@
 <attribute name="NAME" x="107.696" y="65.7225" size="1.27" layer="25" ratio="10" rot="R180"/>
 <attribute name="POPULARITY" value="0" x="106.68" y="66.9925" size="1.778" layer="27" rot="R180" display="off"/>
-<attribute name="TP_SIGNAL_NAME" value="" x="106.68" y="66.9925" size="1.778" layer="27" rot="R180" display="off"/>
 <attribute name="TP_SIGNAL_NAME" value="" x="107.95" y="69.5325" size="1" layer="37" rot="R180"/>
+<attribute name="TP_SIGNAL_NAME" value="" x="106.68" y="66.9925" size="1.778" layer="27" rot="R180" display="off"/>
 <attribute name="VALUE" x="106.68" y="66.9925" size="0.0254" layer="27" rot="R180"/>
 </element>
@@
 <attribute name="NAME" x="149.7965" y="116.84" size="1.27" layer="25" ratio="10"/>
 <attribute name="POPULARITY" value="0" x="153.035" y="119.38" size="1.778" layer="27" rot="R180" display="off"/>
-<attribute name="TP_SIGNAL_NAME" value="" x="153.035" y="119.38" size="1.778" layer="27" rot="R180" display="off"/>
 <attribute name="TP_SIGNAL_NAME" value="" x="154.305" y="121.92" size="1" layer="37" rot="R180"/>
+<attribute name="TP_SIGNAL_NAME" value="" x="153.035" y="119.38" size="1.778" layer="27" rot="R180" display="off"/>
 <attribute name="VALUE" x="153.035" y="119.38" size="0.0254" layer="27" rot="R180"/>
 </element>
@@
 <attribute name="NAME" x="93.726" y="4.7625" size="1.27" layer="25" ratio="10" rot="R180"/>
 <attribute name="POPULARITY" value="0" x="92.075" y="6.35" size="1.778" layer="27" rot="R180" display="off"/>
-<attribute name="TP_SIGNAL_NAME" value="" x="92.075" y="6.35" size="1.778" layer="27" rot="R180" display="off"/>
 <attribute name="TP_SIGNAL_NAME" value="" x="93.345" y="8.89" size="1" layer="37" rot="R180"/>
+<attribute name="TP_SIGNAL_NAME" value="" x="92.075" y="6.35" size="1.778" layer="27" rot="R180" display="off"/>
 <attribute name="VALUE" x="92.075" y="6.35" size="0.0254" layer="27" rot="R180"/>
 </element>
@@
 <attribute name="NAME" x="86.106" y="4.7625" size="1.27" layer="25" ratio="10" rot="R180"/>
 <attribute name="POPULARITY" value="0" x="84.455" y="6.35" size="1.778" layer="27" rot="R180" display="off"/>
-<attribute name="TP_SIGNAL_NAME" value="" x="84.455" y="6.35" size="1.778" layer="27" rot="R180" display="off"/>
 <attribute name="TP_SIGNAL_NAME" value="" x="85.725" y="8.89" size="1" layer="37" rot="R180"/>
+<attribute name="TP_SIGNAL_NAME" value="" x="84.455" y="6.35" size="1.778" layer="27" rot="R180" display="off"/>
 <attribute name="VALUE" x="84.455" y="6.35" size="0.0254" layer="27" rot="R180"/>
 </element>
@@
 <attribute name="NAME" x="89.916" y="4.7625" size="1.27" layer="25" ratio="10" rot="R180"/>
 <attribute name="POPULARITY" value="0" x="88.265" y="6.35" size="1.778" layer="27" rot="R180" display="off"/>
-<attribute name="TP_SIGNAL_NAME" value="" x="88.265" y="6.35" size="1.778" layer="27" rot="R180" display="off"/>
 <attribute name="TP_SIGNAL_NAME" value="" x="89.535" y="8.89" size="1" layer="37" rot="R180"/>
+<attribute name="TP_SIGNAL_NAME" value="" x="88.265" y="6.35" size="1.778" layer="27" rot="R180" display="off"/>
 <attribute name="VALUE" x="88.265" y="6.35" size="0.0254" layer="27" rot="R180"/>
 </element>
@@
 <attribute name="NAME" x="40.7035" y="45.72" size="1.27" layer="25" ratio="10" rot="R180"/>
 <attribute name="POPULARITY" value="0" x="39.6875" y="46.99" size="1.778" layer="27" rot="R180" display="off"/>
-<attribute name="TP_SIGNAL_NAME" value="" x="39.6875" y="46.99" size="1.778" layer="27" rot="R180" display="off"/>
 <attribute name="TP_SIGNAL_NAME" value="" x="40.9575" y="49.53" size="1" layer="37" rot="R180"/>
+<attribute name="TP_SIGNAL_NAME" value="" x="39.6875" y="46.99" size="1.778" layer="27" rot="R180" display="off"/>
 <attribute name="VALUE" x="39.6875" y="46.99" size="0.0254" layer="27" rot="R180"/>
 </element>
@@
 <attribute name="NAME" x="101.219" y="77.7875" size="1.27" layer="25" ratio="10"/>
 <attribute name="POPULARITY" value="0" x="102.87" y="80.645" size="1.778" layer="27" display="off"/>
-<attribute name="TP_SIGNAL_NAME" value="" x="102.87" y="80.645" size="1.778" layer="27" display="off"/>
 <attribute name="TP_SIGNAL_NAME" value="" x="101.6" y="78.105" size="1" layer="37"/>
+<attribute name="TP_SIGNAL_NAME" value="" x="102.87" y="80.645" size="1.778" layer="27" display="off"/>
 <attribute name="VALUE" x="102.87" y="80.645" size="0.0254" layer="27"/>
 </element>
@@
 <attribute name="NAME" x="73.914" y="100.6475" size="1.27" layer="25" ratio="10"/>
 <attribute name="POPULARITY" value="0" x="73.025" y="103.1875" size="1.778" layer="27" display="off"/>
-<attribute name="TP_SIGNAL_NAME" value="" x="73.025" y="103.1875" size="1.778" layer="27" display="off"/>
 <attribute name="TP_SIGNAL_NAME" value="" x="71.755" y="100.6475" size="1" layer="37"/>
+<attribute name="TP_SIGNAL_NAME" value="" x="73.025" y="103.1875" size="1.778" layer="27" display="off"/>
 <attribute name="VALUE" x="73.025" y="103.1875" size="0.0254" layer="27"/>
 </element>
@@
 <attribute name="NAME" x="187.6425" y="55.499" size="1.27" layer="25" ratio="10" rot="R90"/>
 <attribute name="POPULARITY" value="0" x="184.785" y="57.15" size="1.778" layer="27" display="off"/>
-<attribute name="TP_SIGNAL_NAME" value="" x="184.785" y="57.15" size="1.778" layer="27" display="off"/>
 <attribute name="TP_SIGNAL_NAME" value="" x="183.515" y="54.61" size="1" layer="37"/>
+<attribute name="TP_SIGNAL_NAME" value="" x="184.785" y="57.15" size="1.778" layer="27" display="off"/>
 <attribute name="VALUE" x="184.785" y="57.15" size="0.0254" layer="27"/>
 </element>
@@
 <attribute name="NAME" x="32.3215" y="69.85" size="1.27" layer="25" ratio="10"/>
 <attribute name="POPULARITY" value="0" x="33.9725" y="68.58" size="1.778" layer="27" display="off"/>
-<attribute name="TP_SIGNAL_NAME" value="" x="33.9725" y="68.58" size="1.778" layer="27" display="off"/>
 <attribute name="TP_SIGNAL_NAME" value="" x="32.7025" y="66.04" size="1" layer="37"/>
+<attribute name="TP_SIGNAL_NAME" value="" x="33.9725" y="68.58" size="1.778" layer="27" display="off"/>
 <attribute name="VALUE" x="33.9725" y="68.58" size="0.0254" layer="27"/>
 </element>
@@
 <contactref element="D19" pad="C"/>
 <contactref element="D20" pad="A"/>
-<wire x1="9.525" y1="49.53" x2="12.7" y2="49.53" width="0.3048" layer="16"/>
-<wire x1="12.7" y1="49.53" x2="13.335" y2="48.895" width="0.3048" layer="16"/>
-<wire x1="13.335" y1="48.895" x2="13.335" y2="44.45" width="0.3048" layer="16"/>
-<wire x1="13.335" y1="44.45" x2="15.24" y2="42.545" width="0.3048" layer="16"/>
-<wire x1="12.7" y1="52.07" x2="12.7" y2="49.53" width="0.3048" layer="16"/>
+<wire x1="9.525" y1="49.53" x2="12.7" y2="49.53" width="0.6096" layer="16"/>
+<wire x1="12.7" y1="49.53" x2="13.335" y2="48.895" width="0.6096" layer="16"/>
+<wire x1="13.335" y1="48.895" x2="13.335" y2="44.45" width="0.6096" layer="16"/>
+<wire x1="13.335" y1="44.45" x2="15.24" y2="42.545" width="0.6096" layer="16"/>
+<wire x1="12.7" y1="52.07" x2="12.7" y2="49.53" width="0.6096" layer="16"/>
 </signal>
 <signal name="N$43">
@@
 <wire x1="9.525" y1="60.96" x2="9.525" y2="55.88" width="0.6096" layer="16"/>
 <via x="9.525" y="55.88" extent="1-16" drill="0.5"/>
-<wire x1="9.525" y1="55.88" x2="9.525" y2="52.07" width="0.3048" layer="1"/>
+<wire x1="9.525" y1="55.88" x2="9.525" y2="52.07" width="0.6096" layer="1"/>
 </signal>
 <signal name="N$52">
